File: Garden-Soil-MoistureSensor/Garden-Soil-MoistureSensor.kicad_pcb (KiCad board)
At the start: 2 copper layers, 68.6 x 92.7 mm, 11 parts, among them IC1 CD74HC4067M96, IC2 CD74HC4067M96, J1 Conn_01x15, J2 Conn_01x15, J3 Conn_02x15_Odd_Even, U1 1043

Commit message: finished bigger meter fab files ready.
Routing:
- net GND: track 165.9 -> 480.4 mm, vias 0 -> 4
Other:
- board text added: "15 Station Soil Moisture Meter"
- board text added: "BAT +"
- board text added: "BAT -"
- board text added: "Sense1"
- board text added: "Sense12"
- board text added: "Sense13"
- board text added: "Sense14"
- board text added: "Sense15"
- board text added: "Sense2"
- board text added: "Sense3"
- board text added: "Sense4"
- board text added: "https://github.com/TJLTM/Garden-Soil-Moisture-Meter"
Changed lines of the file:
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@@
   (gr_line (start 114.3 138.43) (end 182.88 138.43) (layer "Edge.Cuts") (width 0.1))
   (gr_line (start 182.88 138.43) (end 182.88 45.72) (layer "Edge.Cuts") (width 0.1))
+  (gr_text "Sense13" (at 158.750274 58.8662) (layer "F.SilkS")
+    (effects (font (size 1 1) (thickness 0.15)))
+  )
+  (gr_text "BAT +" (at 133.6962 136.2861) (layer "F.SilkS")
+    (effects (font (size 1 1) (thickness 0.15)))
+  )
+  (gr_text "Sense15" (at 158.750274 53.7862) (layer "F.SilkS")
+    (effects (font (size 1 1) (thickness 0.15)))
+  )
+  (gr_text "BAT -" (at 133.6962 50.199922) (layer "F.SilkS")
+    (effects (font (size 1 1) (thickness 0.15)))
+  )
+  (gr_text "https://github.com/TJLTM/Garden-Soil-Moisture-Meter" (at 148.676829 47.29364) (layer "F.SilkS")
+    (effects (font (size 1 1) (thickness 0.15)))
+  )
+  (gr_text "Sense4" (at 179.908567 81.7262) (layer "F.SilkS")
+    (effects (font (size 1 1) (thickness 0.15)))
+  )
+  (gr_text "15 Station Soil Moisture Meter" (at 152.379722 49.036178) (layer "F.SilkS")
+    (effects (font (size 1 1) (thickness 0.15)))
+  )
+  (gr_text "Sense14" (at 158.750274 56.3262) (layer "F.SilkS")
+    (effects (font (size 1 1) (thickness 0.15)))
+  )
+  (gr_text "Sense12" (at 158.750274 61.4062) (layer "F.SilkS")
+    (effects (font (size 1 1) (thickness 0.15)))
+  )
+  (gr_text "Sense2" (at 179.908567 86.8062) (layer "F.SilkS")
+    (effects (font (size 1 1) (thickness 0.15)))
+  )
+  (gr_text "Sense3" (at 179.908567 84.2662) (layer "F.SilkS")
+    (effects (font (size 1 1) (thickness 0.15)))
+  )
+  (gr_text "Sense1" (at 179.908567 89.3462) (layer "F.SilkS")
+    (effects (font (size 1 1) (thickness 0.15)))
+  )
   (segment (start 153.9334 71.3718) (end 152.7428 70.1812) (width 0.25) (layer "F.Cu") (net 1))
   (segment (start 157.9597 114.5209) (end 159.26 114.5209) (width 0.25) (layer "F.Cu") (net 1))
@@
   (segment (start 151.7927 128.1304) (end 151.9054 128.1304) (width 0.25) (layer "F.Cu") (net 10))
   (segment (start 151.9054 128.1304) (end 156.2989 128.1304) (width 0.25) (layer "F.Cu") (net 10))
+  (segment (start 117.5004 49.53) (end 180.34 49.53) (width 0.25) (layer "F.Cu") (net 10))
   (segment (start 151.0973 118.2147) (end 151.0973 119.1457) (width 0.25) (layer "F.Cu") (net 10))
   (segment (start 155.2828 80.7428) (end 155.2828 86.0236) (width 0.25) (layer "F.Cu") (net 10))
@@
   (segment (start 156.6867 110.4398) (end 156.6867 110.7509) (width 0.25) (layer "F.Cu") (net 10))
   (segment (start 157.9597 128.4909) (end 156.6594 128.4909) (width 0.25) (layer "F.Cu") (net 10))
+  (segment (start 180.34 134.62) (end 117.475 134.62) (width 0.25) (layer "F.Cu") (net 10))
   (segment (start 155.2828 109.0359) (end 156.6867 110.4398) (width 0.25) (layer "F.Cu") (net 10))
   (segment (start 153.8554 113.5822) (end 153.7746 113.5822) (width 0.25) (layer "F.Cu") (net 10))
   (segment (start 151.9054 128.1304) (end 151.9054 119.9538) (width 0.25) (layer "F.Cu") (net 10))
+  (via (at 180.34 49.53) (size 3.8736) (drill 3.175) (layers "F.Cu" "B.Cu") (free) (net 10))
+  (via (at 117.5004 49.53) (size 3.8736) (drill 3.175) (layers "F.Cu" "B.Cu") (free) (net 10))
+  (via (at 180.34 134.62) (size 3.8736) (drill 3.175) (layers "F.Cu" "B.Cu") (free) (net 10))
+  (via (at 117.475 134.62) (size 3.8736) (drill 3.175) (layers "F.Cu" "B.Cu") (free) (net 10))
   (segment (start 174.225 110.3504) (end 174.225 111.5257) (width 0.25) (layer "B.Cu") (net 10))
+  (segment (start 117.5004 134.5946) (end 117.475 134.62) (width 0.25) (layer "B.Cu") (net 10))
   (segment (start 141.5662 56.3333) (end 147.4056 56.3333) (width 0.25) (layer "B.Cu") (net 10))
   (segment (start 174.225 128.4242) (end 175.4003 127.2489) (width 0.25) (layer "B.Cu") (net 10))
   (segment (start 154.1575 72.4318) (end 154.1575 78.4922) (width 0.25) (layer "B.Cu") (net 10))
+  (segment (start 180.34 134.62) (end 180.34 49.53) (width 0.25) (layer "B.Cu") (net 10))
   (segment (start 150.2254 131.8727) (end 171.2153 131.8727) (width 0.25) (layer "B.Cu") (net 10))
   (segment (start 175.4003 127.2489) (end 175.4003 112.3336) (width 0.25) (layer "B.Cu") (net 10))
@@
   (segment (start 148.4151 129.27) (end 149.5547 128.1304) (width 0.25) (layer "B.Cu") (net 10))
   (segment (start 154.1575 78.4922) (end 155.2828 79.6175) (width 0.25) (layer "B.Cu") (net 10))
+  (segment (start 125.8262 64.6933) (end 125.8262 57.8558) (width 0.25) (layer "B.Cu") (net 10))
   (segment (start 147.4056 56.3333) (end 156.2878 65.2155) (width 0.25) (layer "B.Cu") (net 10))
   (segment (start 155.2828 71.3065) (end 154.1575 72.4318) (width 0.25) (layer "B.Cu") (net 10))
@@
   (segment (start 175.4003 112.3336) (end 174.5924 111.5257) (width 0.25) (layer "B.Cu") (net 10))
   (segment (start 155.2828 70.1812) (end 155.2828 71.3065) (width 0.25) (layer "B.Cu") (net 10))
+  (segment (start 125.8262 57.8558) (end 117.5004 49.53) (width 0.25) (layer "B.Cu") (net 10))
+  (segment (start 117.5004 49.53) (end 117.5004 134.5946) (width 0.25) (layer "B.Cu") (net 10))
   (segment (start 148.4151 130.0624) (end 150.2254 131.8727) (width 0.25) (layer "B.Cu") (net 10))
   (segment (start 174.5924 111.5257) (end 174.225 111.5257) (width 0.25) (layer "B.Cu") (net 10))
